File: test_lib.kicad_pcb (KiCad board)
At the start: 2 copper layers, 2 parts, among them J1 CONUFL001-SMD, U1 ESP32-S3-WROOM-1-N8R8

Commit message: initial commit
Parts:
- added U2: MCP1827-ADJE_AT, custom_lib_fp:TO170P1066X482X1572-5, F.Cu at (129.2, 113.6)
Connections:
- U1 pad 2: unconnected-(U1-3V3-Pad2) -> Net-(U1-3V3)
Routing:
- net Net-(U1-3V3): track 0.00 -> 42.9 mm
- net Net-(U2-GND): track 43.1 -> 63.8 mm, vias 0 -> 1
